File: CADENCE BMS Board/Inhibit_System.kicad_sch (KiCad schematic)
At the start: 62 parts, among them IC2 LTC7004IMSE#WTRPBF, IC3 LTC7004IMSE#WTRPBF, IC4 LTC7004IMSE#WTRPBF, IC5 LTC7004IMSE#WTRPBF, IC6 LTC7004IMSE#WTRPBF, J16 INHIBIT_P2, J17 INHIBIT_P2, J18 INHIBIT_P2, J19 INHIBIT_P2, J22 INHIBIT_P2, J23 INHIBIT_P2, J24 INHIBIT_P2, J25 INHIBIT_P2, J26 INHIBIT_P2, Q11 SUD23N06-31-GE3, Q12 SUD23N06-31-GE3, Q13 SUD23N06-31-GE3, Q14 SUD23N06-31-GE3, Q15 SUD23N06-31-GE3, Q16 SUD23N06-31-GE3, Q17 SUD23N06-31-GE3, SW1 SW_SPST, SW2 SW_SPST, SW3 SW_SPST, SW4 SW_SPDT, SW5 SW_SPST, SW6 SW_SPST, SW7 SW_SPST, SW8 SW_SPST, SW9 SW_SPST, U8 MIC4427YM-TR, U9 MIC4427YM-TR

Commit message: Updates to the Inhibit system and Connectors
Other:
- note added: "12.6V"
- moved on the sheet: C33, R46, R47, TP22, TP23

Commit message: Fixed some inhibits
Connections:
- net HIGH_SIDE_PWR: now also IC4.1 (VCC)
Other:
- note added: "Activation inhibit: 3 Feet switches on the top 3 Feet siwtches on the bottom"
- note removed: "Activation inhibit: 2 Feet switches on the top 2 Feet siwtches on the bottom"
- note removed: "https://nepp.nasa.gov/radhome/papers/2020-Topper-NSREC-TID-SEE-Compendium-DW-Paper-20205007136.pdf"
- note removed: "https://nepp.nasa.gov/radhome/papers/CP-2018-OBryan-NSREC-SEE-DW-Paper-20205001490.pdf"

Commit message: Minor Fixes
added test point and output back to solar charger and cleaned up inhibit system a little bit
Other:
- note added: "Place holder for BOM (Foot Switches)"
- note added: "Place holder for BOM (RBF)"
- note added: "Switches for drivers so they don't consume power before deployment"
- note removed: "Place holder for BOM"
- moved on the sheet: J18, J22, SW4
