File: CADENCE BMS Board/Power.kicad_sch (KiCad schematic)
At the start: 60 parts, among them J20 Conn_01x02, U1 TVS2200DRV, U2 LT8612, U3 LT3652IMSE#PBF

Commit message: Removed filters
Solar Charger & Power Regulator
Parts:
- removed C14: 10nF, Capacitor_SMD:C_0805_2012Metric, symbol Device:C
- removed C15: 10uF, Capacitor_SMD:C_1210_3225Metric, symbol Device:C
- removed C16: 4.7uF, Capacitor_SMD:C_1206_3216Metric, symbol Device:C
- removed C39: 10uF, Capacitor_SMD:C_1210_3225Metric, symbol Device:C_Small
- removed C40: 10nF, Capacitor_SMD:C_0805_2012Metric, symbol Device:C_Small
- removed D6: CHG, LED_SMD:LED_0402_1005Metric, symbol Device:LED
- removed FB1: 600, Inductor_SMD:L_1008_2520Metric, symbol Device:FerriteBead_Small
- removed L4: 4.7u, FNR5040S4R7MT:FNR5040S4R7MT, symbol Device:L
- removed R15: 10K, Resistor_SMD:R_1210_3225Metric, symbol Device:R
- removed TP4: Charger-Out, TestPoint:TestPoint_THTPad_D1.0mm_Drill0.5mm, symbol Connector:TestPoint
Connections:
- net at C13.1, R12.1, R14.2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: now also D3.1 (K); no longer D4.1 (A)
- net at D4.2 (K): now also C12.2, U3.11 (BOOST); no longer D3.1 (K)
- new net: D3.2 (A), D4.1 (A)
Other:
- moved on the sheet: D2, D3, D4, R10

Commit message: Minor Fixes
added test point and output back to solar charger and cleaned up inhibit system a little bit
Parts:
- added D6: CHG, LED_SMD:LED_0402_1005Metric, symbol Device:LED
- added R15: 10K, Resistor_SMD:R_1210_3225Metric, symbol Device:R
- added TP4: Charger-Out, TestPoint:TestPoint_THTPad_D1.0mm_Drill0.5mm, symbol Connector:TestPoint
Connections:
- net Cell 1+: now also C13.1, D3.1 (K), R12.1, R14.2, U3.9 (BAT), R15.1, TP4.1
- net VSS: now also D6.1 (K)
- new net: D6.2 (A), R15.2
Other:
- note added: "A rectifying diode (D4) from Bat to boost. Also a 1uF from boost to SW pin.(6) Added series zener (6.1)"
- note removed: "A rectifying diode (D3) from Bat to boost. Also a 1uF from boost to SW pin.(6) Added series zener (6.1)"
