File: CADENCE BMS Board V1/BMS_Board_Prototype.kicad_pcb (KiCad board)
At the start: 4 copper layers, 97 x 97 mm, 191 parts, among them IC1 R5432V407BA, J1 Screw_Terminal_01x02, J10 Conn_01x08, J11 Conn_01x06, J12 Conn_01x02, J13 Conn_01x08, J14 Conn_01x04, J15 Conn_01x08, J2 Conn_01x02, J20 Conn_01x02, J21 Conn_01x02, J27 USB_C_Receptacle_USB2.0_16P, J3 Conn_01x08, J4 Conn_01x02, J5 Conn_01x01_Socket, J6 Conn_01x01_Socket, J7 Conn_01x01_Socket, J8 Conn_01x01_Socket, J9 Conn_01x04, Q1 P-Channel FET, Q10 N-MOS, Q2 60V Enhancement, Q27 Q_PMOS_DGS, Q28 Q_PMOS_DGS, Q3 60V Enhancement, Q4 60V Enhancement, Q5 Q_NMOS_DSG, Q6 Q_NMOS_DSG, Q7 Q_NMOS_DSG, Q8 N-MOS, Q9 N-MOS, U1 TVS2200DRV, U11 CYPD3177-24LQ, U2 LT8612, U3 LT3652IMSE#PBF, U4 BQ34Z100-R2, U5 MCP9600-E_MX, U7 P82B715DR

Commit message: Finalizing updates for V1 of BMS
Parts:
- moved D3 12.6 mm to (37.3, 39.9), turned to 90 degrees
- moved G*** 0.71 mm to (112.0, 76.0)
Connections:
- C12 pad 2: Net-(D3-A) -> Net-(D4-K)
- C13 pad 1: Net-(D4-A) -> Net-(D3-K)
- C14 pad 1: Net-(D4-A) -> Net-(D3-K)
- C15 pad 1: Net-(D4-A) -> Net-(D3-K)
- D4 pad 1: Net-(D4-A) -> Net-(D3-A)
- D4 pad 2: Net-(D3-K) -> Net-(D4-K)
- L4 pad 2: Net-(D4-A) -> Net-(D3-K)
- R12 pad 1: Net-(D4-A) -> Net-(D3-K)
- R14 pad 2: Net-(D4-A) -> Net-(D3-K)
- U3 pad 11: Net-(D3-A) -> Net-(D4-K)
- U3 pad 9: Net-(D4-A) -> Net-(D3-K)
Routing:
- net Cell 3-: track 256.2 -> 389.4 mm
- net Net-(D3-K): track 5.27 -> 72.5 mm, vias 0 -> 2
- net Net-(D4-A): track 62.5 -> 0.00 mm
- net Net-(D4-K): track 0.00 -> 22.3 mm
- net Net-(D3-A): track 12.9 -> 21.7 mm, vias 1 -> 0
- net REG25: track 18.2 -> 17.0 mm, vias 1 -> 0
- net NTC: track 76.9 -> 77.4 mm

Commit message: Cleaning up for BMS V1
Routing:
- net Cell 3-: track 389.4 -> 341.9 mm, vias 94 -> 95
Changed lines of the file:
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@@
+	)
+	(via
+		(at 68 84.5)
+		(size 0.6)
+		(drill 0.3)
+		(layers "F.Cu" "B.Cu")
+		(net "Cell 3-")
 	)
 	(via
@@
 	)
 	(segment
-		(start 69.5 88.6)
-		(end 69.5 87.175)
-		(width 0.2)
-		(layer "B.Cu")
-		(net "Cell 3-")
-	)
-	(segment
 		(start 96.7069 78.4569)
 		(end 96.7069 77.612498)
@@
 	)
 	(segment
-		(start 67.75 83.3)
-		(end 67.75 85.425)
+		(start 67.75 84.75)
+		(end 68 84.5)
 		(width 0.2)
 		(layer "B.Cu")
@@
 	)
 	(segment
-		(start 45.36262 80.059281)
-		(end 61.559281 80.059281)
-		(width 0.2)
-		(layer "B.Cu")
-		(net "Cell 3-")
-	)
-	(segment
 		(start 109.4 88.384744)
 		(end 106.159744 91.625)
@@
 	)
 	(segment
+		(start 67.75 85.425)
+		(end 67.75 84.75)
+		(width 0.2)
+		(layer "B.Cu")
+		(net "Cell 3-")
+	)
+	(segment
 		(start 119.25 56.5)
 		(end 118.75 56)
@@
 	(segment
 		(start 65.75 81.3)
-		(end 67.75 83.3)
-		(width 0.2)
-		(layer "B.Cu")
-		(net "Cell 3-")
-	)
-	(segment
-		(start 64.55 80.1)
-		(end 65.75 81.3)
-		(width 0.781437)
-		(layer "B.Cu")
-		(net "Cell 3-")
-	)
-	(segment
-		(start 65.75 81.3)
 		(end 65.75 80.75)
 		(width 0.2)
@@
 	)
 	(segment
-		(start 69.5 87.175)
-		(end 67.75 85.425)
-		(width 0.2)
-		(layer "B.Cu")
-		(net "Cell 3-")
-	)
-	(segment
-		(start 63.5 80.1)
-		(end 64.55 80.1)
-		(width 0.781437)
-		(layer "B.Cu")
-		(net "Cell 3-")
-	)
-	(segment
 		(start 81.25 66.025)
 		(end 79.475 64.25)
@@
 	)
 	(segment
-		(start 34.394401 91.0275)
-		(end 45.36262 80.059281)
-		(width 0.2)
-		(layer "B.Cu")
-		(net "Cell 3-")
-	)
-	(segment
 		(start 96.5 79)
 		(end 96.4138 78.9138)
 		(width 0.2)
 		(layer "B.Cu")
-		(net "Cell 3-")
-	)
-	(segment
-		(start 29.2 91.0275)
-		(end 34.394401 91.0275)
-		(width 0.2)
-		(layer "B.Cu")
