File: CADENCE BMS Board V1/BMS_Board_Prototype.kicad_pcb (KiCad board)
At the start: 4 copper layers, 97 x 97 mm, 188 parts, among them IC1 R5432V407BA, J1 Screw_Terminal_01x02, J10 Conn_01x08, J11 Conn_01x06, J12 Conn_01x02, J13 Conn_01x08, J14 Conn_01x04, J15 Conn_01x08, J2 Conn_01x02, J20 Conn_01x02, J21 Conn_01x02, J27 USB_C_Receptacle_USB2.0_16P, J28 Conn_01x02, J29 Conn_01x02, J3 Conn_01x08, J30 Conn_01x02, J31 Conn_01x04, J4 Conn_01x02, J5 Conn_01x01_Socket, J6 Conn_01x01_Socket, J7 Conn_01x01_Socket, J8 Conn_01x01_Socket, J9 Conn_01x04, Q1 P-Channel FET, Q10 N-MOS, Q2 60V Enhancement, Q27 Q_PMOS_DGS, Q28 Q_PMOS_DGS, Q3 60V Enhancement, Q4 60V Enhancement, Q5 Q_NMOS_DSG, Q6 Q_NMOS_DSG, Q7 Q_NMOS_DSG, Q8 N-MOS, Q9 N-MOS, U1 TVS2200DRV, U11 CYPD3177-24LQ, U2 LT8612, U3 LT3652IMSE#PBF, U4 BQ34Z100-R2, U5 MCP9600-E_MX, U7 P82B715DR

Commit message: Updates to finalize V1
Parts:
- moved J28 81.5 mm to (60.2, 35.0)
- moved J31 78.6 mm to (51.5, 59.0)
- moved R49 7.50 mm to (53.5, 53.0)
- moved G*** 7.27 mm to (32.5, 46.0)
- moved R12 4.60 mm to (53.5, 50.5)
- moved R50 2.26 mm to (51.0, 51.5)
- moved G*** 2.21 mm to (97.0, 34.8)
Connections:
- C1 pad 2: VSS -> Solar1-
- C11 pad 1: VSS -> Solar1-
- C13 pad 2: VSS -> Solar1-
- C17 pad 2: VSS -> Solar1-
- C18 pad 1: VSS -> Solar1-
- C19 pad 1: VSS -> Solar1-
- C2 pad 1: VSS -> Solar1-
- C20 pad 1: VSS -> Solar1-
- C22 pad 1: VSS -> Solar1-
- C23 pad 1: VSS -> Solar1-
- C24 pad 1: VSS -> Solar1-
- C25 pad 2: VSS -> Solar1-
- C26 pad 1: VSS -> Solar1-
- C3 pad 1: VSS -> Solar1-
- C31 pad 2: VSS -> Solar1-
- C32 pad 2: VSS -> Solar1-
- C4 pad 2: VSS -> Solar1-
- C41 pad 2: VSS -> Solar1-
- C42 pad 2: VSS -> Solar1-
- C43 pad 2: VSS -> Solar1-
- C5 pad 2: VSS -> Solar1-
- C55 pad 2: VSS -> Solar1-
- C57 pad 1: VSS -> Solar1-
- C59 pad 2: VSS -> Solar1-
- C6 pad 2: VSS -> Solar1-
- C60 pad 2: VSS -> Solar1-
- C61 pad 2: VSS -> Solar1-
- C7 pad 2: VSS -> Solar1-
- C9 pad 1: VSS -> Solar1-
- D15 pad 2: VSS -> Solar1-
- D2 pad 1: VSS -> Solar1-
- D5 pad 1: VSS -> Solar1-
- D6 pad 1: VSS -> Solar1-
- D7 pad 2: VSS -> Solar1-
- D9 pad 2: VSS -> Solar1-
- IC1 pad 9: VSS -> Solar1-
- J10 pad 4: VSS -> Solar1-
- J12 pad 2: VSS -> Solar1-
- J13 pad 4: VSS -> Solar1-
- J15 pad 4: VSS -> Solar1-
- J2 pad 2: VSS -> Solar1-
- J20 pad 2: VSS -> Solar1-
- J27 pad A1: VSS -> Solar1-
- J27 pad A12: VSS -> Solar1-
- J27 pad B1: VSS -> Solar1-
- J27 pad B12: VSS -> Solar1-
- J27 pad SH: VSS -> Solar1-
- J29 pad 2: VSS -> Solar1-
- J3 pad 4: VSS -> Solar1-
- J30 pad 2: VSS -> Solar1-
- J31 pad 4: VSS -> Solar1-
- J4 pad 2: VSS -> Solar1-
- J9 pad 2: VSS -> Solar1-
- J9 pad 4: VSS -> Solar1-
- Q3 pad 2: VSS -> Solar1-
- Q4 pad 2: VSS -> Solar1-
- Q5 pad 2: VSS -> Solar1-
- R1 pad 2: VSS -> Solar1-
- R13 pad 2: VSS -> Solar1-
- R20 pad 2: VSS -> Solar1-
- R31 pad 1: VSS -> Solar1-
- R4 pad 2: VSS -> Solar1-
- R59 pad 2: VSS -> Solar1-
- R71 pad 2: VSS -> Solar1-
- R9 pad 2: VSS -> Solar1-
- TP6 pad 1: VSS -> Solar1-
- U1 pad 1: VSS -> Solar1-
- U1 pad 2: VSS -> Solar1-
- U1 pad 3: VSS -> Solar1-
- U1 pad 7: VSS -> Solar1-
- U11 pad 19: VSS -> Solar1-
- U11 pad 22: VSS -> Solar1-
- U11 pad 25: VSS -> Solar1-
- U11 pad 6: VSS -> Solar1-
- U2 pad 10: VSS -> Solar1-
- U2 pad 11: VSS -> Solar1-
- U2 pad 12: VSS -> Solar1-
- U2 pad 13: VSS -> Solar1-
- U2 pad 14: VSS -> Solar1-
- U2 pad 29: VSS -> Solar1-
- U2 pad 8: VSS -> Solar1-
- U2 pad 9: VSS -> Solar1-
- U3 pad 13: VSS -> Solar1-
- U3 pad 6: VSS -> Solar1-
- U4 pad 1: VSS -> Solar1-
- U4 pad 8: VSS -> Solar1-
- U5 pad 1: VSS -> Solar1-
- U5 pad 10: VSS -> Solar1-
- U5 pad 13: VSS -> Solar1-
- U5 pad 16: VSS -> Solar1-
- U5 pad 17: VSS -> Solar1-
- U5 pad 18: VSS -> Solar1-
- U5 pad 21: VSS -> Solar1-
- U5 pad 3: VSS -> Solar1-
- U5 pad 5: VSS -> Solar1-
- U5 pad 6: VSS -> Solar1-
- U5 pad 7: VSS -> Solar1-
- U5 pad 9: VSS -> Solar1-
- U7 pad 4: VSS -> Solar1-
Routing:
- net Solar1-: track 72.3 -> 289.9 mm, vias 0 -> 77
- net VSS: track 169.9 -> 0.00 mm, vias 82 -> 0
- net (no net): track 55.3 -> 0.00 mm, vias 2 -> 0
- net V_mppt_o: track 1.55 -> 49.2 mm, vias 1 -> 2
- net Cell 1+: track 181.3 -> 198.4 mm, vias 15 -> 5
- net Cell 3-: track 118.6 -> 135.5 mm, vias 13 -> 6
- net V_mppt_i: track 0.00 -> 10.3 mm
- net +3.3V: track 164.2 -> 156.3 mm
- net HS_I2C1_LDA: track 65.5 -> 68.4 mm
- net CB3: track 28.5 -> 31.2 mm, vias 0 -> 2
- net Solar Power: track 149.2 -> 151.4 mm
- net Net-(R49-Pad2): track 3.98 -> 1.95 mm
- net Net-(R12-Pad2): track 3.80 -> 2.02 mm
- net Net-(Q6-G): track 26.7 -> 25.9 mm
- net UNREG: track 13.2 -> 13.8 mm, vias 11 -> 17
- added copper zone on B.Cu, net Cell 3-
- added copper zone on B.Cu, net Solar1-
- added copper zone on In1.Cu, net Solar1-
- removed copper zone on F.Cu, net Cell 1+
- removed copper zone on B.Cu, net VSS
- removed copper zone on In1.Cu, net VSS
Other:
- board text added: "Inhibit CON"
- board text added: "USB PWR"

Commit message: Updates for connector footprint
Parts:
- added G***: LOGO, LOGO, F.Cu at (79.5, 46.0)
- J14: footprint Connector_JST:JST_NV_B04P-NV_1x04_P5.00mm_Vertical -> Connector_Samtec_HPM_THT:Samtec_HPM-04-05-x-S_Straight_1x04_Pitch5.08mm
- moved J9 0.47 mm to (56.5, 71.5)
- moved J14 0.23 mm to (29.0, 106.1), turned to 180 degrees
Routing:
- net +3.3V: track 156.3 -> 152.9 mm
Other:
- board text added: "LAUGH"
- board text added: "LIVE"
- board text added: "LOVE"

Commit message: Final Changes for Manufacturing
Routing:
- net +3.3V: track 152.9 -> 152.2 mm
Changed lines of the file:
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@@
-	)
-	(segment
-		(start 48.94375 83.29375)
-		(end 48.94375 87.153568)
-		(width 0.781437)
-		(layer "F.Cu")
-		(net "+3.3V")
 	)
 	(segment
@@
 	)
 	(segment
-		(start 60.7625 71.475)
-		(end 60.440718 71.796782)
-		(width 0.781437)
-		(layer "F.Cu")
-		(net "+3.3V")
-	)
-	(segment
 		(start 91.627274 83.302974)
 		(end 91.481796 83.302974)
@@
 	)
 	(segment
+		(start 48.94375 84.03125)
+		(end 48.94375 87.153568)
+		(width 0.781437)
+		(layer "F.Cu")
+		(net "+3.3V")
+	)
+	(segment
 		(start 52.627177 91.2375)
 		(end 53.669468 92.279791)
@@
 		(start 59.2 89.75)
 		(end 59.2 95.75)
+		(width 0.781437)
+		(layer "F.Cu")
+		(net "+3.3V")
+	)
+	(segment
+		(start 48.94375 84.03125)
+		(end 61.5 71.475)
 		(width 0.781437)
 		(layer "F.Cu")
@@
 	)
 	(segment
-		(start 61.5 71.475)
-		(end 60.7625 71.475)
-		(width 0.781437)
-		(layer "F.Cu")
-		(net "+3.3V")
-	)
-	(segment
 		(start 53.669468 92.279791)
 		(end 53.669468 93.295209)
@@
 		(end 82.266246 84.25)
 		(width 0.2)
-		(layer "F.Cu")
-		(net "+3.3V")
-	)
-	(segment
-		(start 60.440718 72.196765)
-		(end 59.596765 73.040718)
-		(width 0.781437)
-		(layer "F.Cu")
-		(net "+3.3V")
-	)
-	(segment
-		(start 59.196782 73.040718)
-		(end 48.94375 83.29375)
-		(width 0.781437)
 		(layer "F.Cu")
 		(net "+3.3V")
@@
 	)
 	(segment
-		(start 60.440718 71.796782)
-		(end 60.440718 72.196765)
-		(width 0.781437)
-		(layer "F.Cu")
-		(net "+3.3V")
-	)
-	(segment
-		(start 61.5 71)
-		(end 61.475 71)
-		(width 0.781437)
-		(layer "F.Cu")
-		(net "+3.3V")
-	)
-	(segment
 		(start 84.553992 81.89439)
 		(end 82.232314 84.216068)
@@
 		(layer "F.Cu")
 		(net "+3.3V")
-	)
-	(segment
-		(start 59.596765 73.040718)
-		(end 59.196782 73.040718)
-		(width 0.781437)
-		(layer "F.Cu")
-		(net "+3.3V")
