File: CADENCE BMS Board V1/I2C_Components.kicad_sch (KiCad schematic)
At the start: 11 parts, among them U7 P82B715DR

Commit message: Removed 3v3Q
Removed 3v3Q, Capacitors (EMI FILTER OUT), Changed all +3.3V Q -> 3.3V
Connections:
- net +3.3V Q renamed +3.3V
Changed lines of the file:
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@@
 			)
 		)
-		(property "Value" "+3.3V Q"
+		(property "Value" "+3.3V"
 			(at 129.54 63.5 0)
 			(show_name no)
@@
 			)
 		)
-		(property "Value" "+3.3V Q"
+		(property "Value" "+3.3V"
 			(at 83.82 54.61 0)
 			(show_name no)
@@
 			)
 		)
-		(property "Value" "+3.3V Q"
+		(property "Value" "+3.3V"
 			(at 107.95 54.61 0)
 			(show_name no)
@@
 			)
 		)
-		(property "Value" "+3.3V Q"
+		(property "Value" "+3.3V"
 			(at 146.05 63.5 0)
 			(show_name no)
