File: CADENCE BMS Board V1/Inhibit_System.kicad_sch (KiCad schematic)
At the start: 62 parts, among them IC2 LTC7004IMSE#WTRPBF, IC3 LTC7004IMSE#WTRPBF, IC4 LTC7004IMSE#WTRPBF, IC5 LTC7004IMSE#WTRPBF, IC6 LTC7004IMSE#WTRPBF, J16 INHIBIT_P2, J17 INHIBIT_P2, J18 INHIBIT_P2, J19 INHIBIT_P2, J22 INHIBIT_P2, J23 INHIBIT_P2, J24 INHIBIT_P2, J25 INHIBIT_P2, J26 INHIBIT_P2, Q11 SUD23N06-31-GE3, Q12 SUD23N06-31-GE3, Q13 SUD23N06-31-GE3, Q14 SUD23N06-31-GE3, Q15 SUD23N06-31-GE3, Q16 SUD23N06-31-GE3, Q17 SUD23N06-31-GE3, SW1 SW_SPST, SW2 SW_SPST, SW3 SW_SPST, SW4 SW_SPDT, SW5 SW_SPST, SW6 SW_SPST, SW7 SW_SPST, SW8 SW_SPST, SW9 SW_SPST, U8 MIC4427YM-TR, U9 MIC4427YM-TR

Commit message: Cleaning up the Schematic
Other:
- note added: "Gate Driver Switches"
- moved on the sheet: J18, J22
Changed lines of the file:
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@@
 	(paper "A3")
 	(rectangle
+		(start 339.09 93.98)
+		(end 386.08 118.11)
+		(stroke
+			(width 0)
+			(type default)
+		)
+		(fill
+			(type none)
+		)
+	)
+	(rectangle
 		(start 120.65 180.34)
 		(end 262.89 220.98)
@@
 		)
 	)
+	(text "Gate Driver Switches\n"
+		(exclude_from_sim no)
+		(at 361.188 121.158 0)
+		(effects
+			(font
+				(size 2.54 2.54)
+				(thickness 0.508)
+				(bold yes)
+				(color 0 255 6 1)
+			)
+		)
+	)
 	(text "Goes back in Vin \nof Solar Charger\nto prevent V_mppt\ngoing into UNREG\n"
 		(exclude_from_sim no)
@@
 	(wire
 		(pts
-			(xy 365.76 107.95) (xy 365.76 110.49)
+			(xy 367.03 107.95) (xy 367.03 110.49)
 		)
 		(stroke
@@
 	(wire
 		(pts
-			(xy 353.06 101.6) (xy 353.06 104.14)
+			(xy 354.33 101.6) (xy 354.33 104.14)
 		)
 		(stroke
@@
 	(wire
 		(pts
-			(xy 353.06 107.95) (xy 353.06 110.49)
+			(xy 354.33 107.95) (xy 354.33 110.49)
 		)
 		(stroke
@@
 	(wire
 		(pts
-			(xy 365.76 101.6) (xy 365.76 104.14)
+			(xy 367.03 101.6) (xy 367.03 104.14)
 		)
 		(stroke
@@
 	(global_label "HIGH_SIDE_PWR"
 		(shape input)
-		(at 365.76 109.22 0)
+		(at 367.03 109.22 0)
 		(fields_autoplaced yes)
 		(effects
@@
 		)
 		(property "Intersheetrefs" "${INTERSHEET_REFS}"
-			(at 383.4409 109.22 0)
+			(at 384.7109 109.22 0)
 			(hide yes)
 			(show_name no)
@@
 	(global_label "LOW_SIDE_PWR"
 		(shape input)
-		(at 365.76 102.87 0)
+		(at 367.03 102.87 0)
 		(fields_autoplaced yes)
 		(effects
@@
 		)
 		(property "Intersheetrefs" "${INTERSHEET_REFS}"
-			(at 382.7151 102.87 0)
+			(at 383.9851 102.87 0)
 			(hide yes)
 			(show_name no)
@@
 	(global_label "Cell 1+"
 		(shape input)
-		(at 353.06 102.87 180)
+		(at 354.33 102.87 180)
 		(fields_autoplaced yes)
 		(effects
@@
 		)
 		(property "Intersheetrefs" "${INTERSHEET_REFS}"
-			(at 342.6363 102.87 0)
+			(at 343.9063 102.87 0)
 			(hide yes)
 			(show_name no)
@@
 	(global_label "Cell 1+"
 		(shape input)
-		(at 353.06 109.22 180)
+		(at 354.33 109.22 180)
 		(fields_autoplaced yes)
 		(effects
@@
 		)
 		(property "Intersheetrefs" "${INTERSHEET_REFS}"
-			(at 342.6363 109.22 0)
+			(at 343.9063 109.22 0)
 			(hide yes)
 			(show_name no)
@@
 	(symbol
 		(lib_id "Connector_Generic:Conn_02x02_Odd_Even")
-		(at 358.14 101.6 0)
+		(at 359.41 101.6 0)
 		(unit 1)
 		(body_style 1)
@@
 		(fields_autoplaced yes)
 		(property "Reference" "J18"
-			(at 359.41 95.25 0)
+			(at 360.68 95.25 0)
 			(show_name no)
 			(do_not_autoplace no)
@@
 		)
 		(property "Value" "INHIBIT_P2"
-			(at 359.41 97.79 0)
+			(at 360.68 97.79 0)
 			(show_name no)
 			(do_not_autoplace no)
@@
 		)
 		(property "Footprint" "Connector_Hirose:Hirose_DF11-4DP-2DSA_2x02_P2.00mm_Vertical"
-			(at 358.14 101.6 0)
+			(at 359.41 101.6 0)
 			(hide yes)
 			(show_name no)
@@
 		)
 		(property "Datasheet" ""
-			(at 358.14 101.6 0)
+			(at 359.41 101.6 0)
 			(hide yes)
 			(show_name no)
@@
 		)
 		(property "Description" "Generic connector, double row, 02x02, odd/even pin numbering scheme (row 1 odd numbers, row 2 even numbers), script generated (kicad-library-utils/schlib/autogen/connector/)"
-			(at 358.14 101.6 0)
+			(at 359.41 101.6 0)
 			(hide yes)
 			(show_name no)
@@
 		)
 		(property "LCSC" ""
-			(at 358.14 101.6 0)
+			(at 359.41 101.6 0)
 			(hide yes)
 			(show_name no)
@@
 		)
 		(property "Sim.Type" ""
-			(at 358.14 101.6 0)
+			(at 359.41 101.6 0)
 			(hide yes)
 			(show_name no)
@@
 		)
 		(property "Voltage" ""
-			(at 358.14 101.6 0)
+			(at 359.41 101.6 0)
 			(hide yes)
 			(show_name no)
@@
 	(symbol
 		(lib_id "Connector_Generic:Conn_02x02_Odd_Even")
-		(at 358.14 107.95 0)
+		(at 359.41 107.95 0)
 		(unit 1)
 		(body_style 1)
@@
 		(dnp no)
 		(property "Reference" "J22"
-			(at 359.664 113.538 0)
+			(at 360.934 113.538 0)
 			(show_name no)
 			(do_not_autoplace no)
@@
 		)
 		(property "Value" "INHIBIT_P2"
-			(at 359.664 116.078 0)
+			(at 360.934 116.078 0)
 			(show_name no)
 			(do_not_autoplace no)
@@
 		)
 		(property "Footprint" "Connector_Hirose:Hirose_DF11-4DP-2DSA_2x02_P2.00mm_Vertical"
-			(at 358.14 107.95 0)
+			(at 359.41 107.95 0)
 			(hide yes)
 			(show_name no)
@@
 		)
 		(property "Datasheet" ""
-			(at 358.14 107.95 0)
+			(at 359.41 107.95 0)
 			(hide yes)
 			(show_name no)
@@
 		)
 		(property "Description" "Generic connector, double row, 02x02, odd/even pin numbering scheme (row 1 odd numbers, row 2 even numbers), script generated (kicad-library-utils/schlib/autogen/connector/)"
-			(at 358.14 107.95 0)
+			(at 359.41 107.95 0)
 			(hide yes)
 			(show_name no)
@@
 		)
 		(property "LCSC" ""
-			(at 358.14 107.95 0)
+			(at 359.41 107.95 0)
 			(hide yes)
 			(show_name no)
@@
 		)
 		(property "Sim.Type" ""
-			(at 358.14 107.95 0)
+			(at 359.41 107.95 0)
 			(hide yes)
 			(show_name no)
@@
 		)
 		(property "Voltage" ""
-			(at 358.14 107.95 0)
+			(at 359.41 107.95 0)
 			(hide yes)
 			(show_name no)
