File: CADENCE BMS Board V1/Sensor.kicad_sch (KiCad schematic)
At the start: 65 parts, among them IC1 R5432V407BA, J1 Screw_Terminal_01x02, J21 Conn_01x02, Q1 P-Channel FET, Q10 N-MOS, Q2 60V Enhancement, Q3 60V Enhancement, Q4 60V Enhancement, Q5 Q_NMOS_DSG, Q6 Q_NMOS_DSG, Q7 Q_NMOS_DSG, Q8 N-MOS, Q9 N-MOS, U4 BQ34Z100-R2, U5 MCP9600-E_MX

Commit message: Removed 3v3Q
Removed 3v3Q, Capacitors (EMI FILTER OUT), Changed all +3.3V Q -> 3.3V
Connections:
- net +3.3V Q renamed +3.3V
Changed lines of the file:
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@@
 			)
 		)
-		(property "Value" "+3.3V Q"
+		(property "Value" "+3.3V"
 			(at 166.37 255.2699 0)
 			(show_name no)

Commit message: New connectors and adding in a test setup
Connections:
- net Cell 1+: no longer Q1.2 (S), Q2.3 (D), R16.1, R17.1, R35.1, TP5.1, TP8.1
- new net UNREG: Q1.2 (S), Q2.3 (D), R16.1, R17.1, R35.1, TP5.1, TP8.1
Changed lines of the file:
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@@
 		)
 	)
-	(global_label "Cell 1+"
+	(global_label "UNREG"
 		(shape input)
 		(at 433.07 66.04 0)
@@
 		)
 		(property "Intersheetrefs" "${INTERSHEET_REFS}"
-			(at 443.4937 66.04 0)
+			(at 442.4052 66.04 0)
 			(hide yes)
 			(show_name no)
@@
 		)
 	)
-	(global_label "Cell 1+"
+	(global_label "UNREG"
 		(shape input)
 		(at 38.1 127 180)
@@
 		)
 		(property "Intersheetrefs" "${INTERSHEET_REFS}"
-			(at 27.6763 127 0)
-			(hide yes)
-			(show_name no)
+			(at 28.7648 127 0)
+			(hide yes)
+			(show_name no)

Commit message: Updates to component testing
Changed lines of the file:
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@@
 	(text "These diode are in case of overvoltage they will\ntake the hit instead of the buffer or the IC"
 		(exclude_from_sim no)
-		(at 160.274 92.964 0)
+		(at 154.686 85.852 0)
 		(effects
 			(font
-				(size 0.635 0.635)
+				(size 1.27 1.27)
 				(thickness 0.127)
 				(bold yes)
