File: CADENCE Inhibit System Test Board/CADENCE Inhibit System Test Board.kicad_sch (KiCad schematic)
At the start: 62 parts, among them IC2 LTC7004IMSE#WTRPBF, IC3 LTC7004IMSE#WTRPBF, IC4 LTC7004IMSE#WTRPBF, IC5 LTC7004IMSE#WTRPBF, IC6 LTC7004IMSE#WTRPBF, J16 INHIBIT_P2, J17 INHIBIT_P2, J18 INHIBIT_P2, J19 INHIBIT_P2, J22 INHIBIT_P2, J23 INHIBIT_P2, J24 INHIBIT_P2, J25 INHIBIT_P2, J26 INHIBIT_P2, Q11 SUD23N06-31-GE3, Q12 SUD23N06-31-GE3, Q13 SUD23N06-31-GE3, Q14 SUD23N06-31-GE3, Q15 SUD23N06-31-GE3, Q16 SUD23N06-31-GE3, Q17 SUD23N06-31-GE3, SW1 SW_SPST, SW2 SW_SPST, SW3 SW_SPST, SW4 SW_SPDT, SW5 SW_SPST, SW6 SW_SPST, SW7 SW_SPST, SW8 SW_SPST, SW9 SW_SPST, U8 MIC4427YM-TR, U9 MIC4427YM-TR

Commit message: Updated reference designators for Inhibit System
Automatically updated ref designators
Parts:
- renumbered C44 to C1, C34 to C10, C46 to C2, C45 to C3, C47 to C4, C33 to C5, C37 to C6, C38 to C7, C35 to C8, C36 to C9, D11 to D1, D12 to D2, D13 to D3, D14 to D4, D16 to D5, D17 to D6, IC5 to IC1, IC6 to IC2, IC2 to IC5, J23 to J1, J24 to J2, J16 to J3, J26 to J4, J17 to J5, J25 to J6, J19 to J7, J18 to J8, J22 to J9, Q13 to Q1, Q14 to Q2, Q17 to Q3, Q15 to Q4, Q16 to Q5, Q11 to Q6, Q12 to Q7, R60 to R1, R51 to R10, R48 to R11, R61 to R2, R55 to R3, R56 to R4, R46 to R5, R47 to R6, R52 to R7, R53 to R8, R54 to R9, SW5 to SW2, SW8 to SW3, SW2 to SW5, SW9 to SW7, SW3 to SW8, SW7 to SW9, TP22 to TP1, TP23 to TP2, TP21 to TP3, U8 to U1, U9 to U2
Other:
- note added: "Enable Switches for FET Drivers"
- note added: "Example Referece, External RBF pin that will need connectors"
- note added: "Max: 12.435V Nom: 10.8V"
- note added: "Place holder for BOM (Feet Switches)"
- note added: "Place holder for BOM (RBF)"
- note removed: "External RBF pin that will need connectors"
- note removed: "Max: 12.6V Nom: 10.8V"
- note removed: "Place holder for BOM"
- note removed: "https://nepp.nasa.gov/radhome/papers/2020-Topper-NSREC-TID-SEE-Compendium-DW-Paper-20205007136.pdf"
- note removed: "https://nepp.nasa.gov/radhome/papers/CP-2018-OBryan-NSREC-SEE-DW-Paper-20205001490.pdf"
- moved on the sheet: J8, J9, SW4

Commit message: Updating footprint glitch
Parts:
- D1, D2, D3, D4: footprint MMBD914LT1G Diode:SOT-23_ONS -> MMBD914LT1G_Diode:SOT-23_ONS
- IC1, IC2, IC3, IC4, IC5: footprint LTC7004IMSE#WTRPBF_Gate_Driver:MSE_05-08-1664_ADI -> LTC7004IMSE#WTRPBF Gate Driver:MSE_05-08-1664_ADI

Commit message: bms connectors
Parts:
- added J10: Conn_01x04, Connector_JST:JST_XH_B4B-XH-A_1x04_P2.50mm_Vertical, symbol Connector_Generic:Conn_01x04
- added J11: Conn_01x02, Connector_JST:JST_XH_B2B-XH-A_1x02_P2.50mm_Vertical, symbol Connector_Generic:Conn_01x02
- added TP4: TestPoint, symbol Connector:TestPoint
Connections:
- net Cell 1+: now also J10.1 (Pin_1)
- net Cell 3-: now also J10.3 (Pin_3)
- net UNREG: now also J10.2 (Pin_2)
- net VSS: now also J10.4 (Pin_4)
- net V_mppt_i: now also J11.2 (Pin_2)
- net V_mppt_o: now also J11.1 (Pin_1)
- net at D3.1 (K), D4.1 (K), J1.1 (Pin_1)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: now also TP4.1
Other:
- note added: "BMS Connections"

Commit message: test points added
Parts:
- added TP6, TP7: TestPoint, symbol Connector:TestPoint
Connections:
- net Cell 3-: now also TP6.1
- net VSS: now also TP7.1
Changed lines of the file:
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@@
 	)
 	(junction
+		(at 115.57 102.87)
+		(diameter 0)
+		(color 0 0 0 0)
+	)
+	(junction
 		(at 205.74 193.04)
 		(diameter 0)
@@
 	)
 	(junction
+		(at 115.57 165.1)
+		(diameter 0)
+		(color 0 0 0 0)
+	)
+	(junction
 		(at 215.9 193.04)
 		(diameter 0)
@@
 	(wire
 		(pts
-			(xy 115.57 99.06) (xy 115.57 106.68)
+			(xy 115.57 99.06) (xy 115.57 102.87)
 		)
 		(stroke
@@
 	(wire
 		(pts
+			(xy 115.57 102.87) (xy 115.57 106.68)
+		)
+		(stroke
+			(width 0)
+			(type default)
+		)
+	)
+	(wire
+		(pts
 			(xy 205.74 74.93) (xy 205.74 76.2)
 		)
@@
 	(wire
 		(pts
-			(xy 115.57 157.48) (xy 115.57 167.64)
+			(xy 115.57 157.48) (xy 115.57 165.1)
 		)
 		(stroke
@@
 	(wire
 		(pts
+			(xy 115.57 165.1) (xy 115.57 167.64)
+		)
+		(stroke
+			(width 0)
+			(type default)
+		)
+	)
+	(wire
+		(pts
 			(xy 120.65 63.5) (xy 120.65 72.39)
 		)
@@
 	)
 	(symbol
+		(lib_id "Connector:TestPoint")
+		(at 115.57 102.87 270)
+		(unit 1)
+		(body_style 1)
+		(exclude_from_sim no)
+		(in_bom yes)
+		(on_board yes)
+		(in_pos_files yes)
+		(dnp no)
+		(fields_autoplaced yes)
+		(property "Reference" "TP6"
+			(at 120.65 101.5999 90)
+			(show_name no)
+			(do_not_autoplace no)
+			(effects
+				(font
+					(size 1.27 1.27)
+				)
+				(justify left)
+			)
+		)
+		(property "Value" "TestPoint"
+			(at 120.65 104.1399 90)
+			(show_name no)
+			(do_not_autoplace no)
+			(effects
+				(font
+					(size 1.27 1.27)
+				)
+				(justify left)
+			)
+		)
+		(property "Footprint" ""
+			(at 115.57 107.95 0)
+			(hide yes)
+			(show_name no)
+			(do_not_autoplace no)
+			(effects
+				(font
+					(size 1.27 1.27)
+				)
+			)
+		)
+		(property "Datasheet" ""
+			(at 115.57 107.95 0)
+			(hide yes)
+			(show_name no)
+			(do_not_autoplace no)
+			(effects
+				(font
+					(size 1.27 1.27)
+				)
+			)
+		)
+		(property "Description" "test point"
+			(at 115.57 102.87 0)
+			(hide yes)
+			(show_name no)
+			(do_not_autoplace no)
+			(effects
+				(font
+					(size 1.27 1.27)
+				)
+			)
+		)
+		(pin "1"
+		)
+		(instances
+			(project "CADENCE Inhibit System Test Board"
+				(path "/191bd9c3-424d-41a4-b898-2e1885f219ad"
+					(reference "TP6")
+					(unit 1)
+				)
+			)
+		)
+	)
+	(symbol
 		(lib_id "Switch:SW_SPST")
 		(at 381 90.17 0)
@@
 					(unit 1)
 				)
+			)
+		)
+	)
+	(symbol
+		(lib_id "Connector:TestPoint")
+		(at 115.57 165.1 270)
+		(unit 1)
+		(body_style 1)
+		(exclude_from_sim no)
+		(in_bom yes)
+		(on_board yes)
+		(in_pos_files yes)
+		(dnp no)
+		(fields_autoplaced yes)
+		(property "Reference" "TP7"
+			(at 120.65 163.8299 90)
+			(show_name no)
+			(do_not_autoplace no)
+			(effects
+				(font
+					(size 1.27 1.27)
+				)
+				(justify left)
+			)
+		)
+		(property "Value" "TestPoint"
+			(at 120.65 166.3699 90)
+			(show_name no)
+			(do_not_autoplace no)
+			(effects
+				(font
+					(size 1.27 1.27)
+				)
+				(justify left)
+			)
+		)
+		(property "Footprint" ""
+			(at 115.57 170.18 0)
+			(hide yes)
+			(show_name no)
+			(do_not_autoplace no)
+			(effects
+				(font
+					(size 1.27 1.27)
+				)
+			)
+		)
+		(property "Datasheet" ""
+			(at 115.57 170.18 0)
+			(hide yes)
+			(show_name no)
+			(do_not_autoplace no)
+			(effects
+				(font
+					(size 1.27 1.27)
+				)
+			)
+		)
+		(property "Description" "test point"
+			(at 115.57 165.1 0)
+			(hide yes)
+			(show_name no)
+			(do_not_autoplace no)
+			(effects
+				(font
+					(size 1.27 1.27)
+				)
+			)
+		)
+		(pin "1"
+		)
+		(instances
+			(project "CADENCE Inhibit System Test Board"
+				(path "/191bd9c3-424d-41a4-b898-2e1885f219ad"
+					(reference "TP7")
+					(unit 1)
+				)

Commit message: test points added
Parts:
- added TP5: UNREG, symbol Connector:TestPoint
- added TP8: V_mppt_o, symbol Connector:TestPoint
- added TP9: V_mppt_i, symbol Connector:TestPoint
- TP4: value TestPoint -> Voltage Level
- TP6: value TestPoint -> Cell 3-
- TP7: value TestPoint -> VSS
Connections:
- net UNREG: now also TP5.1
- net V_mppt_i: now also TP9.1
- net V_mppt_o: now also TP8.1
Other:
- moved on the sheet: TP4, TP6
