File: CADENCE Inhibit System Test Board/CADENCE Inhibit System Test Board.kicad_sch (KiCad schematic)
At the start: 70 parts, among them IC1 LTC7004IMSE#WTRPBF, IC2 LTC7004IMSE#WTRPBF, IC3 LTC7004IMSE#WTRPBF, IC4 LTC7004IMSE#WTRPBF, IC5 LTC7004IMSE#WTRPBF, J1 INHIBIT_P2, J10 Conn_01x04, J11 Conn_01x02, J2 INHIBIT_P2, J3 INHIBIT_P2, J4 INHIBIT_P2, J5 INHIBIT_P2, J6 INHIBIT_P2, J7 INHIBIT_P2, J8 INHIBIT_P2, J9 INHIBIT_P2, Q1 SUD23N06-31-GE3, Q2 SUD23N06-31-GE3, Q3 SUD23N06-31-GE3, Q4 SUD23N06-31-GE3, Q5 SUD23N06-31-GE3, Q6 SUD23N06-31-GE3, Q7 SUD23N06-31-GE3, SW1 SW_SPST, SW2 SW_SPST, SW3 SW_SPST, SW4 SW_SPDT, SW5 SW_SPST, SW6 SW_SPST, SW7 SW_SPST, SW8 SW_SPST, SW9 SW_SPST, U1 MIC4427YM-TR, U2 MIC4427YM-TR

Commit message: mounting holes added
Parts:
- added H1, H2, H3, H4: MountingHole, MountingHole:MountingHole_3.2mm_M3, symbol Mechanical:MountingHole
Other:
- note added: "MOUNTING HOLES"

Commit message: moved parts and updated mounting holes
Parts:
- removed H1, H2, H3, H4: MountingHole, MountingHole:MountingHole_3.2mm_M3, symbol Mechanical:MountingHole
- added H1, H2, H3, H4: MountingHole_Pad, MountingHole:MountingHole_3.2mm_M3_DIN965_Pad_TopOnly, symbol Mechanical:MountingHole_Pad

Commit message: updated schematic
Connections:
- net VSS: now also H1.1, H2.1, H3.1, H4.1
Changed lines of the file:
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@@
 	)
 	(junction
+		(at 353.06 160.02)
+		(diameter 0)
+		(color 0 0 0 0)
+	)
+	(junction
 		(at 224.79 166.37)
 		(diameter 0)
@@
 	)
 	(junction
+		(at 353.06 172.72)
+		(diameter 0)
+		(color 0 0 0 0)
+	)
+	(junction
 		(at 115.57 140.97)
 		(diameter 0)
@@
 	)
 	(junction
+		(at 353.06 166.37)
+		(diameter 0)
+		(color 0 0 0 0)
+	)
+	(junction
 		(at 224.79 93.98)
 		(diameter 0)
@@
 	(wire
 		(pts
+			(xy 353.06 172.72) (xy 353.06 179.07)
+		)
+		(stroke
+			(width 0)
+			(type default)
+		)
+	)
+	(wire
+		(pts
 			(xy 143.51 198.12) (xy 143.51 199.39)
 		)
@@
 	(wire
 		(pts
+			(xy 378.46 160.02) (xy 353.06 160.02)
+		)
+		(stroke
+			(width 0)
+			(type default)
+		)
+	)
+	(wire
+		(pts
 			(xy 102.87 60.96) (xy 102.87 59.69)
 		)
@@
 	(wire
 		(pts
+			(xy 378.46 153.67) (xy 353.06 153.67)
+		)
+		(stroke
+			(width 0)
+			(type default)
+		)
+	)
+	(wire
+		(pts
 			(xy 205.74 40.64) (xy 205.74 41.91)
 		)
@@
 	(wire
 		(pts
+			(xy 353.06 172.72) (xy 378.46 172.72)
+		)
+		(stroke
+			(width 0)
+			(type default)
+		)
+	)
+	(wire
+		(pts
 			(xy 97.79 152.4) (xy 106.68 152.4)
 		)
@@
 	(wire
 		(pts
+			(xy 353.06 166.37) (xy 353.06 172.72)
+		)
+		(stroke
+			(width 0)
+			(type default)
+		)
+	)
+	(wire
+		(pts
 			(xy 115.57 59.69) (xy 120.65 59.69)
 		)
@@
 	(wire
 		(pts
+			(xy 353.06 166.37) (xy 378.46 166.37)
+		)
+		(stroke
+			(width 0)
+			(type default)
+		)
+	)
+	(wire
+		(pts
 			(xy 158.75 199.39) (xy 158.75 198.12)
 		)
@@
 	(wire
 		(pts
+			(xy 353.06 153.67) (xy 353.06 160.02)
+		)
+		(stroke
+			(width 0)
+			(type default)
+		)
+	)
+	(wire
+		(pts
+			(xy 353.06 160.02) (xy 353.06 166.37)
+		)
+		(stroke
+			(width 0)
+			(type default)
+		)
+	)
+	(wire
+		(pts
 			(xy 91.44 91.44) (xy 100.33 91.44)
 		)
@@
 					(unit 1)
 				)
+			)
+		)
+	)
+	(symbol
+		(lib_id "power:GND")
+		(at 353.06 179.07 0)
+		(unit 1)
+		(body_style 1)
+		(exclude_from_sim no)
+		(in_bom yes)
+		(on_board yes)
+		(in_pos_files yes)
+		(dnp no)
+		(property "Reference" "#PWR018"
+			(at 353.06 185.42 0)
+			(hide yes)
+			(show_name no)
+			(do_not_autoplace no)
+			(effects
+				(font
+					(size 1.27 1.27)
+				)
+			)
+		)
+		(property "Value" "VSS"
+			(at 355.6 179.578 0)
+			(show_name no)
+			(do_not_autoplace no)
+			(effects
+				(font
+					(size 1.27 1.27)
+				)
+			)
+		)
+		(property "Footprint" ""
+			(at 353.06 179.07 0)
+			(hide yes)
+			(show_name no)
+			(do_not_autoplace no)
+			(effects
+				(font
+					(size 1.27 1.27)
+				)
+			)
+		)
+		(property "Datasheet" ""
+			(at 353.06 179.07 0)
+			(hide yes)
+			(show_name no)
+			(do_not_autoplace no)
+			(effects
+				(font
+					(size 1.27 1.27)
+				)
+			)
+		)
+		(property "Description" "Power symbol creates a global label with name \"GND\" , ground"
+			(at 353.06 179.07 0)
+			(hide yes)
+			(show_name no)
+			(do_not_autoplace no)
+			(effects
+				(font
+					(size 1.27 1.27)
+				)
+			)
+		)
+		(pin "1"
+		)
+		(instances
+			(project "CADENCE Inhibit System Test Board"
+				(path "/191bd9c3-424d-41a4-b898-2e1885f219ad"
+					(reference "#PWR018")
+					(unit 1)
+				)

Commit message: value name change
Parts:
- R6: value 100k -> 100K
Changed lines of the file:
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@@
 			)
 		)
-		(property "Value" "100k"
+		(property "Value" "100K"
 			(at 134.62 71.1199 0)
 			(show_name no)

Commit message: fixed diode footprints and added gbr and drl files
Connections:
- net Cell 1+: now also D2.1 (A); no longer D2.2 (A)
- net V_mppt_i: now also D1.1 (A); no longer D1.2 (A)
- net at J1.1 (Pin_1), J1.3 (Pin_3), J2.1 (Pin_1)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: now also D3.3 (K), D4.3 (K); no longer D3.1 (K), D4.1 (K)
- new net: D1.3 (K), D3.1 (A)
- new net: D2.3 (K), D4.1 (A)
Changed lines of the file:
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@@
 	)
 	(symbol
+		(lib_name "1N914_1")
 		(lib_id "Diode:1N914")
 		(at 46.99 57.15 180)
@@
 		(pin "1"
 		)
-		(pin "2"
+		(pin "3"
 		)
 		(instances
@@
 	)
 	(symbol
+		(lib_name "1N914_3")
 		(lib_id "Diode:1N914")
 		(at 46.99 74.93 180)
@@
 		(pin "1"
 		)
-		(pin "2"
+		(pin "3"
 		)
 		(instances
@@
 	)
 	(symbol
+		(lib_name "1N914_2")
 		(lib_id "Diode:1N914")
 		(at 59.69 57.15 180)
@@
 		(pin "1"
 		)
-		(pin "2"
+		(pin "3"
 		)
 		(instances
@@
 		(pin "1"
 		)
-		(pin "2"
+		(pin "3"
 		)
 		(instances
