File: CADENCE Inhibit System Test Board/CADENCE Inhibit System Test Board.kicad_pcb (KiCad board)
At the start: 2 copper layers, 70 x 72.5 mm, 65 parts, among them IC1 LTC7004IMSE#WTRPBF, IC2 LTC7004IMSE#WTRPBF, IC3 LTC7004IMSE#WTRPBF, IC4 LTC7004IMSE#WTRPBF, IC5 LTC7004IMSE#WTRPBF, J1 INHIBIT_P2, J10 Conn_01x04, J11 Conn_01x02, J2 INHIBIT_P2, J3 INHIBIT_P2, J4 INHIBIT_P2, J5 INHIBIT_P2, J6 INHIBIT_P2, J7 INHIBIT_P2, J8 INHIBIT_P2, J9 INHIBIT_P2, Q1 SUD23N06-31-GE3, Q2 SUD23N06-31-GE3, Q3 SUD23N06-31-GE3, Q4 SUD23N06-31-GE3, Q5 SUD23N06-31-GE3, Q6 SUD23N06-31-GE3, Q7 SUD23N06-31-GE3, U1 MIC4427YM-TR, U2 MIC4427YM-TR

Commit message: edited mosfet traces
Parts:
- moved TP3 2.86 mm to (182.0, 80.8)
- moved H3 0.72 mm to (184.0, 104.4)
- moved TP5 0.60 mm to (170.2, 103.2)
Routing:
- net Net-(IC1-TGDN): track 16.3 -> 13.4 mm
- net Net-(IC2-TS): track 40.1 -> 41.7 mm
- net Cell 3-: track 34.2 -> 35.4 mm, vias 0 -> 1
- net LOW_SIDE_PWR: track 68.0 -> 68.6 mm
- net EN: track 162.2 -> 162.7 mm
- net UNREG: track 81.0 -> 80.9 mm, vias 2 -> 4
