File: CADENCE Solar Board/Solar Board/Solar Board.kicad_sch (KiCad schematic)
At the start: 20 parts, among them J1 Conn_01x08, U1 INA230AIRGTT, U2 AD7414ARTZ-1REEL7, U3 OPT3001IDNPRQ1

Commit message: PCB updates
added custom solar cell footprints and created base layer for the thin PCB board
Other:
- note added: "Light Sensor"
- note removed: "Light Sensor (Double check ADDR pin connection)"
Changed lines of the file:
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@@
 		)
 	)
-	(text "Light Sensor (Double check ADDR pin connection)\n\n\n"
+	(text "Light Sensor\n\n\n"
 		(exclude_from_sim no)
-		(at 155.702 20.828 0)
+		(at 151.638 21.59 0)
 		(effects
 			(font
