File: CADENCE Solar Board/Solar Board 8s2p/Solar Board.kicad_pcb (KiCad board)
At the start: 2 copper layers, 100 x 351 mm, 28 parts, among them J1 Conn_01x08, U1 INA230AIRGTT, U2 AD7414ARTZ-1REEL7, U3 OPT3001IDNPRQ1

Commit message: added separate project folders
8sp1 and 8sp2 are identical except for the pcb layout. solar cells are added to the 8s2p version. traces added to the pcb, had to be moved because of a previous height issue.
Parts:
- added SC: CAVU Solar Cell, Solar Cell Library:CAVU Solar Cell, F.Cu at (212.5, 232.0)
- added SC: CAVU Solar Cell, Solar Cell Library:CAVU Solar Cell, F.Cu at (212.5, 152.0)
- added SC: CAVU Solar Cell, Solar Cell Library:CAVU Solar Cell, F.Cu at (212.4, 72.0)
- added SC: CAVU Solar Cell, Solar Cell Library:CAVU Solar Cell, F.Cu at (126.2, 142.0)
- added SC: CAVU Solar Cell, Solar Cell Library:CAVU Solar Cell, F.Cu at (126.2, 302.0)
- added SC: CAVU Solar Cell, Solar Cell Library:CAVU Solar Cell, F.Cu at (126.2, 222.0)
- added SC: CAVU Solar Cell, Solar Cell Library:CAVU Solar Cell, F.Cu at (126.2, 61.9)
- added SC: CAVU Solar Cell, Solar Cell Library:CAVU Solar Cell, F.Cu at (212.5, 312.0)
- moved TP3 8.86 mm to (61.5, 32.5)
- moved TP2 6.73 mm to (82.5, 30.5)
- moved SC 2.54 mm to (111.0, 317.5)
- moved SC 2.54 mm to (111.0, 237.5)
- moved SC 2.54 mm to (110.9, 77.5)
- moved SC 2.54 mm to (111.0, 157.5)
- moved SC 2.54 mm to (24.7, 67.3)
- moved SC 2.54 mm to (24.8, 147.5)
- moved SC 2.54 mm to (24.8, 227.5)
- moved SC 2.54 mm to (24.8, 307.5)
- moved J1 2.48 mm to (80.0, 37.5)
- moved TP1 1.12 mm to (85.0, 34.5)
Routing:
- net Solar1-: track 4.98 -> 14.6 mm, vias 0 -> 1
- net Solar1+: track 18.0 -> 26.0 mm, vias 0 -> 2
- net HS_I2C1_LCL: track 27.9 -> 33.2 mm
- net HS_I2C1_LDA: track 37.9 -> 35.7 mm
- net GND: track 1.44 -> 0.89 mm
Other:
- board size 100 x 351 mm -> 206 x 340.4 mm

Commit message: Updates
removed light sensor, changed pcb design, added screw holes for 8s1p and 8s2p configurations, optimized via paths in pcb
Parts:
- removed C1: 100nF, Capacitor_SMD:C_0805_2012Metric
- removed R8: 10k, Resistor_SMD:R_0805_2012Metric
- removed the SC at (212.5, 232.0)
- removed the SC at (212.5, 152.0)
- removed the SC at (212.4, 72.0)
- removed the SC at (126.2, 142.0)
- removed the SC at (126.2, 302.0)
- removed the SC at (126.2, 222.0)
- removed the SC at (126.2, 61.9)
- removed the SC at (212.5, 312.0)
- removed U3: OPT3001IDNPRQ1, OPT3001IDNPRQ1:SON65P200X200X65-7N-D
- added REF**: MountingHole_3.2mm_M3, MountingHole:MountingHole_3.2mm_M3, F.Cu at (103.0, 93.0)
- added REF**: MountingHole_3.2mm_M3, MountingHole:MountingHole_3.2mm_M3, F.Cu at (52.2, 4.50)
- added REF**: MountingHole_3.2mm_M3, MountingHole:MountingHole_3.2mm_M3, F.Cu at (153.8, 4.50)
- added REF**: MountingHole_3.2mm_M3, MountingHole:MountingHole_3.2mm_M3, F.Cu at (103.0, 257.4)
- added REF**: MountingHole_3.2mm_M3, MountingHole:MountingHole_3.2mm_M3, F.Cu at (153.8, 335.9)
- added REF**: MountingHole_3.2mm_M3, MountingHole:MountingHole_3.2mm_M3, F.Cu at (52.2, 335.9)
- added SC: CAVU Solar Cell, Solar Cell Library:CAVU Solar Cell, F.Cu at (114.7, 290.0)
- added SC: CAVU Solar Cell, Solar Cell Library:CAVU Solar Cell, F.Cu at (201.0, 300.0)
- added SC: CAVU Solar Cell, Solar Cell Library:CAVU Solar Cell, F.Cu at (200.9, 60.0)
- added SC: CAVU Solar Cell, Solar Cell Library:CAVU Solar Cell, F.Cu at (114.7, 130.0)
- added SC: CAVU Solar Cell, Solar Cell Library:CAVU Solar Cell, F.Cu at (114.7, 49.8)
- added SC: CAVU Solar Cell, Solar Cell Library:CAVU Solar Cell, F.Cu at (201.0, 140.0)
- added SC: CAVU Solar Cell, Solar Cell Library:CAVU Solar Cell, F.Cu at (114.7, 210.0)
- added SC: CAVU Solar Cell, Solar Cell Library:CAVU Solar Cell, F.Cu at (201.0, 220.0)
- moved C3 33.4 mm to (38.6, 8.09)
- moved C2 32.4 mm to (43.0, 6.62), turned to 0 degrees
- moved U2 28.8 mm to (40.3, 3.44)
- moved R5 28.5 mm to (34.8, 6.68)
- moved D2 27.8 mm to (31.0, 3.67)
- moved R7 27.3 mm to (47.4, 2.19)
- moved R6 27.1 mm to (35.0, 3.96)
- moved R1 25.3 mm to (62.4, 9.03)
- moved R4 25.3 mm to (58.9, 9.03)
- moved D1 24.6 mm to (41.2, 11.1)
- moved SC 24.6 mm to (93.7, 220.0)
- moved SC 24.6 mm to (93.7, 300.0)
- moved SC 24.6 mm to (93.7, 140.0)
- moved SC 24.6 mm to (7.42, 130.0)
- moved SC 24.6 mm to (7.42, 210.0)
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Routing:
- net GND: track 0.89 -> 12.7 mm, vias 0 -> 7
- net +3.3V: track 0.00 -> 6.66 mm
- net HS_I2C1_LDA: track 35.7 -> 29.1 mm, vias 5 -> 2
- net Net-(U2-AS): track 3.67 -> 5.63 mm, vias 0 -> 2
- net Solar1+: track 26.0 -> 27.8 mm, vias 2 -> 0
- net Net-(U1-V_S+): track 2.37 -> 4.00 mm
- net Net-(U3-INT): track 1.59 -> 0.00 mm
- net Net-(U2-ALERT): track 7.62 -> 6.13 mm
- net Net-(U1-ALERT): track 7.58 -> 8.76 mm
- net HS_I2C1_LCL: track 33.2 -> 32.1 mm, vias 2 -> 4
- net Solar1-: track 14.6 -> 13.7 mm, vias 1 -> 4
- net Net-(D2-A): track 1.96 -> 2.54 mm
