File: CADENCE BMS Board V2/Power.kicad_sch (KiCad schematic)
At the start: 62 parts, among them J20 Conn_01x02, J28 Banana Socket PWR, J29 Banana Socket VSS, U1 TVS2200DRV, U2 LT8612, U3 LT3652IMSE#PBF

Commit message: Updates for banana plug power testing
Parts:
- removed J28: Banana Socket PWR, Connector:Banana_Cliff_FCR7350R_S16N-PC_Horizontal, symbol Connector:Conn_01x01_Socket
- removed J29: Banana Socket VSS, Connector:Banana_Cliff_FCR7350B_S16N-PC_Horizontal, symbol Connector:Conn_01x01_Socket
Connections:
- net VDC_OUT: now reaches D18.2 (A)
Changed lines of the file:
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@@
 	(wire
 		(pts
-			(xy 78.74 46.99) (xy 102.87 46.99)
-		)
-		(stroke
-			(width 0)
-			(type default)
-		)
-	)
-	(wire
-		(pts
 			(xy 124.46 331.47) (xy 124.46 337.82)
 		)
@@
 	(wire
 		(pts
-			(xy 77.47 36.83) (xy 82.55 36.83)
-		)
-		(stroke
-			(width 0)
-			(type default)
-		)
-	)
-	(wire
-		(pts
 			(xy 316.23 63.5) (xy 323.85 63.5)
 		)
@@
 	(wire
 		(pts
+			(xy 99.06 46.99) (xy 102.87 46.99)
+		)
+		(stroke
+			(width 0)
+			(type default)
+		)
+	)
+	(wire
+		(pts
 			(xy 256.54 48.26) (xy 256.54 46.99)
 		)
@@
 		)
 	)
+	(global_label "VDC_OUT"
+		(shape input)
+		(at 99.06 46.99 180)
+		(fields_autoplaced yes)
+		(effects
+			(font
+				(size 1.27 1.27)
+			)
+			(justify right)
+		)
+		(property "Intersheetrefs" "${INTERSHEET_REFS}"
+			(at 87.85 46.99 0)
+			(hide yes)
+			(show_name no)
+			(do_not_autoplace no)
+			(effects
+				(font
+					(size 1.27 1.27)
+				)
+				(justify right)
+			)
+		)
+	)
 	(global_label "FAULT'"
 		(shape input)
@@
 	)
 	(symbol
-		(lib_id "Connector:Conn_01x01_Socket")
-		(at 73.66 46.99 180)
-		(unit 1)
-		(body_style 1)
-		(exclude_from_sim no)
-		(in_bom yes)
-		(on_board yes)
-		(in_pos_files yes)
-		(dnp no)
-		(fields_autoplaced yes)
-		(property "Reference" "J28"
-			(at 74.295 41.91 0)
-			(show_name no)
-			(do_not_autoplace no)
-			(effects
-				(font
-					(size 1.27 1.27)
-				)
-			)
-		)
-		(property "Value" "Banana Socket PWR"
-			(at 74.295 44.45 0)
-			(show_name no)
-			(do_not_autoplace no)
-			(effects
-				(font
-					(size 1.27 1.27)
-				)
-			)
-		)
-		(property "Footprint" "Connector:Banana_Cliff_FCR7350R_S16N-PC_Horizontal"
-			(at 73.66 46.99 0)
-			(hide yes)
-			(show_name no)
-			(do_not_autoplace no)
-			(effects
-				(font
-					(size 1.27 1.27)
-				)
-			)
-		)
-		(property "Datasheet" ""
-			(at 73.66 46.99 0)
-			(hide yes)
-			(show_name no)
-			(do_not_autoplace no)
-			(effects
-				(font
-					(size 1.27 1.27)
-				)
-			)
-		)
-		(property "Description" "Generic connector, single row, 01x01, script generated"
-			(at 73.66 46.99 0)
-			(hide yes)
-			(show_name no)
-			(do_not_autoplace no)
-			(effects
-				(font
-					(size 1.27 1.27)
-				)
-			)
-		)
-		(pin "1"
-		)
-		(instances
-			(project "BMS_Board_Prototype"
-				(path "/4ee99911-836b-4752-8a2d-327c8b28dc47/f4fcff51-0cdb-4e70-aba0-d567fd3e6a03"
-					(reference "J28")
-					(unit 1)
-				)
-			)
-		)
-	)
-	(symbol
 		(lib_id "Device:C")
 		(at 341.63 71.12 0)
@@
 	)
 	(symbol
-		(lib_id "power:GND")
-		(at 82.55 36.83 0)
-		(unit 1)
-		(body_style 1)
-		(exclude_from_sim no)
-		(in_bom yes)
-		(on_board yes)
-		(in_pos_files yes)
-		(dnp no)
-		(property "Reference" "#PWR033"
-			(at 82.55 43.18 0)
-			(hide yes)
-			(show_name no)
-			(do_not_autoplace no)
-			(effects
-				(font
-					(size 1.27 1.27)
-				)
-			)
-		)
-		(property "Value" "VSS"
-			(at 81.28 41.656 0)
-			(show_name no)
-			(do_not_autoplace no)
-			(effects
-				(font
-					(size 1.27 1.27)
-				)
-				(justify left)
-			)
-		)
-		(property "Footprint" ""
-			(at 82.55 36.83 0)
-			(hide yes)
-			(show_name no)
-			(do_not_autoplace no)
-			(effects
-				(font
-					(size 1.27 1.27)
-				)
-			)
-		)
-		(property "Datasheet" ""
-			(at 82.55 36.83 0)
-			(hide yes)
-			(show_name no)
-			(do_not_autoplace no)
-			(effects
-				(font
-					(size 1.27 1.27)
-				)
-			)
-		)
-		(property "Description" "Power symbol creates a global label with name \"GND\" , ground"
-			(at 82.55 36.83 0)
-			(hide yes)
-			(show_name no)
-			(do_not_autoplace no)
-			(effects
-				(font
-					(size 1.27 1.27)
-				)
-			)
-		)
-		(pin "1"
-		)
-		(instances
-			(project "BMS_Board_Prototype"
-				(path "/4ee99911-836b-4752-8a2d-327c8b28dc47/f4fcff51-0cdb-4e70-aba0-d567fd3e6a03"
-					(reference "#PWR033")
-					(unit 1)
-				)
-			)
-		)
-	)
-	(symbol
 		(lib_id "Device:C_Small")
 		(at 100.33 320.04 0)
@@
 					(unit 1)
 				)
-			)
-		)
-	)
-	(symbol
-		(lib_id "Connector:Conn_01x01_Socket")
-		(at 72.39 36.83 180)
-		(unit 1)
-		(body_style 1)
-		(exclude_from_sim no)
-		(in_bom yes)
-		(on_board yes)
-		(in_pos_files yes)
-		(dnp no)
-		(fields_autoplaced yes)
-		(property "Reference" "J29"
-			(at 73.025 31.75 0)
-			(show_name no)
-			(do_not_autoplace no)
-			(effects
-				(font
-					(size 1.27 1.27)
-				)
-			)
-		)
-		(property "Value" "Banana Socket VSS"
-			(at 73.025 34.29 0)
-			(show_name no)
-			(do_not_autoplace no)
-			(effects
-				(font
-					(size 1.27 1.27)
-				)
-			)
-		)
-		(property "Footprint" "Connector:Banana_Cliff_FCR7350B_S16N-PC_Horizontal"
-			(at 72.39 36.83 0)
-			(hide yes)
-			(show_name no)
-			(do_not_autoplace no)
-			(effects
-				(font
-					(size 1.27 1.27)
-				)
-			)
-		)
-		(property "Datasheet" ""
-			(at 72.39 36.83 0)
-			(hide yes)
-			(show_name no)
-			(do_not_autoplace no)
-			(effects
-				(font
-					(size 1.27 1.27)
-				)
-			)
-		)
-		(property "Description" "Generic connector, single row, 01x01, script generated"
-			(at 72.39 36.83 0)
-			(hide yes)
-			(show_name no)
-			(do_not_autoplace no)
-			(effects
-				(font
-					(size 1.27 1.27)
-				)
-			)
-		)
-		(pin "1"
-		)
-		(instances
-			(project "BMS_Board_Prototype"
-				(path "/4ee99911-836b-4752-8a2d-327c8b28dc47/f4fcff51-0cdb-4e70-aba0-d567fd3e6a03"
-					(reference "J29")
-					(unit 1)
-				)

Commit message: Adding in BMS V2 file for editing
Parts:
- removed C14: 10nF, Capacitor_SMD:C_0805_2012Metric, symbol Device:C
- removed C15: 10uF, Capacitor_SMD:C_1210_3225Metric, symbol Device:C
- removed C16: 4.7uF, Capacitor_SMD:C_1206_3216Metric, symbol Device:C
- removed C39: 10uF, Capacitor_SMD:C_1210_3225Metric, symbol Device:C_Small
- removed C40: 10nF, Capacitor_SMD:C_0805_2012Metric, symbol Device:C_Small
- removed FB1: 600, Inductor_SMD:L_1008_2520Metric, symbol Device:FerriteBead_Small
- removed L4: 4.7u, FNR5040S4R7MT:FNR5040S4R7MT, symbol Device:L
- added D20, D21: D_Schottky 40v, Diode_SMD:D_SMA, symbol Device:D_Schottky
- R12, R49, R50: footprint Resistor_SMD:R_2512_6332Metric -> Resistor_SMD:R_0603_1608Metric
Connections:
- net Cell 1+: now also C13.1, D3.1 (K), R12.1, R14.2, U3.9 (BAT); no longer C41.1, L5.1, TP1.1
- net VDC_OUT: now also D20.2 (A); no longer D18.2 (A)
- net at C4.1, C5.1, D18.1 (K)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: now also D20.1 (K), D21.1 (K)
- net V_mppt_o: now reaches C7.1, R3.1, TP2.1, U3.1 (VIN)
- net V_mppt_o: no longer C6.1, R2.2
- new net TEST_PWR: D18.2 (A)
- new net UNREG: C41.1, L5.1, TP1.1
- new net USB PWR: D21.2 (A)
- new net V_mppt_i: C6.1, R2.2
Other:
- note added: "Possible mistake with power good this need a pull up resistor connected to 3.3V in order to send a high signal to MCU be sure to add in next revision"
- note added: "Possibly connect SHDN into the Vin line for next revison if it works on testing so the solar charger can power on without needing 3V3 buck to bypass inhibit system"
- note added: "Removed 3v3Q, Capacitors (EMI FILTER OUT)"
- note added: "The voltage for CHG' and FAULT' are .4V"
- note added: "The voltage for SHDN' is 1.2V nom with (+/-) .5V"
- note added: "These pins need to be activated in order for the IC to output correctly"
- moved on the sheet: D18, D19, D6, R15, TP4
